Commit message: fix bug of torso control link

File: R1/urdf/R1.urdf (robot description, URDF)
Before this commit: robot R1, 30 links, 29 joints
Joints:
- joint torso_joint1: limit lower=-1.1345 upper=1.8326 effort=0 velocity=0 -> lower=-1.1345 upper=1.8326 effort=100 velocity=2.5
- joint torso_joint2: limit lower=-2.7925 upper=2.5307 effort=0 velocity=0 -> lower=-2.7925 upper=2.5307 effort=100 velocity=2.5
- joint torso_joint3: axis 0 0 1 -> 0 0 -1; limit lower=-2.0944 upper=1.8326 effort=0 velocity=0 -> lower=-2.0944 upper=1.8326 effort=100 velocity=2.5
- joint torso_joint4: limit lower=-3.0543 upper=3.0543 effort=0 velocity=0 -> lower=-3.0543 upper=3.0543 effort=100 velocity=2.5
