Commit message: A1XY URDF update

File: A1X/urdf/a1x.urdf (robot description, URDF)
Before this commit: robot a1x, 10 links, 9 joints
Links:
- link gripper_finger_link1: mass 0.020196517310345 -> 0.027
- link gripper_finger_link2: mass 0.0201965174144991 -> 0.027

File: A1Y/urdf/a1y.urdf (robot description, URDF)
Before this commit: robot a1y, 10 links, 9 joints
Links:
- link gripper_finger_link1: mass 0.0201965308906806 -> 0.027
- link gripper_finger_link2: mass 0.0201965308906567 -> 0.027
- link gripper_link: mass 0.246251128080965 -> 0.604
