Commit message: effort velocity update

File: A1Z/A1Z_Flange/urdf/A1Z_Flange.urdf (robot description, URDF)
Before this commit: robot A1Z_Flange, 7 links, 6 joints
Joints:
- joint arm_joint1: limit lower=-2.094 upper=2.094 effort=0 velocity=0 -> lower=-2.094 upper=2.094 effort=20 velocity=5.65
- joint arm_joint2: limit lower=0 upper=3.142 effort=0 velocity=0 -> lower=0 upper=3.142 effort=25 velocity=5.65
- joint arm_joint3: limit lower=0 upper=3.142 effort=0 velocity=0 -> lower=-3.142 upper=0 effort=20 velocity=5.65
- joint arm_joint4: limit lower=-1.309 upper=1.309 effort=0 velocity=0 -> lower=-1.309 upper=1.309 effort=9 velocity=3.77
- joint arm_joint5: limit lower=-1.484 upper=1.484 effort=0 velocity=0 -> lower=-1.484 upper=1.484 effort=3.5 velocity=10.47
- joint arm_joint6: limit lower=-2.007 upper=2.007 effort=0 velocity=0 -> lower=-2.007 upper=2.007 effort=3.5 velocity=10.47

File: A1Z/A1Z_G1Z/urdf/A1Z_G1Z.urdf (robot description, URDF)
Before this commit: robot A1Z_G1Z, 9 links, 8 joints
Joints:
- joint arm_joint1: limit lower=-2.094 upper=2.094 effort=0 velocity=0 -> lower=-2.094 upper=2.094 effort=20 velocity=5.65
- joint arm_joint2: limit lower=0 upper=3.142 effort=0 velocity=0 -> lower=0 upper=3.142 effort=25 velocity=5.65
- joint arm_joint3: limit lower=-3.142 upper=0 effort=0 velocity=0 -> lower=-3.142 upper=0 effort=20 velocity=5.65
- joint arm_joint4: limit lower=-1.309 upper=1.309 effort=0 velocity=0 -> lower=-1.309 upper=1.309 effort=9 velocity=3.77
- joint arm_joint5: limit lower=-1.484 upper=1.484 effort=0 velocity=0 -> lower=-1.484 upper=1.484 effort=3.5 velocity=10.47
- joint arm_joint6: limit lower=-2.007 upper=2.007 effort=0 velocity=0 -> lower=-2.007 upper=2.007 effort=3.5 velocity=10.47
- joint gripper_finger_left_joint: axis 0 1 0 -> (none); limit lower=0 upper=0.048 effort=0 velocity=0 -> (none); type prismatic -> fixed
- joint gripper_finger_rIght_joint: axis 0 1 0 -> (none); limit lower=-0.048 upper=0 effort=0 velocity=0 -> (none); mimic joint=gripper_finger_left_joint multiplier=-1 offset=0 -> (none); type prismatic -> fixed
