Commit message: Update A1Z G1Z model and clean macOS metadata

File: A1Z/A1Z_G1Z/urdf/A1Z_G1Z.urdf (robot description, URDF)
Before this commit: robot A1Z_G1Z, 9 links, 8 joints
Links:
- link arm_link6: mass 0.55665538 -> 0.64400562
- link gripper_finger_left_link: mass 0.13786800 -> 0.14648590
- link gripper_finger_rIght_link: mass 0.13786800 ->  0.14648224
Joints:
- joint gripper_finger_left_joint: axis (none) -> 0 1 0; limit (none) -> lower=0 upper=0.048 effort=3 velocity=10.47; type fixed -> prismatic
- joint gripper_finger_rIght_joint: axis (none) -> 0 1 0; limit (none) -> lower=-0.048 upper=0 effort=3 velocity=10.47; mimic (none) -> joint=gripper_finger_left_joint multiplier=-1 offset=0; type fixed -> prismatic
